Commit message: Successfully converted block to usd to test

File: libs/robot_description/tesollo_DG3F/tesollo_DG3F.urdf (robot description, URDF)
Before this commit: robot delto_gripper_3f, 16 links, 15 joints
Links:
- link F1_01: geometry collision mesh filename=meshes/link_01.stl; visual mesh filename=meshes/link_01.stl
- link F1_02: geometry collision mesh filename=meshes/link_02.stl; visual mesh filename=meshes/link_02.stl
- link F1_03: geometry collision mesh filename=meshes/link_03.stl; visual mesh filename=meshes/link_03.stl
- link F1_04: geometry collision mesh filename=meshes/link_04.stl; visual mesh filename=meshes/link_04.stl
- link F1_TIP: geometry collision mesh filename=meshes/link_tip_high.stl; visual mesh filename=meshes/link_tip_high.stl
- link F2_01: geometry collision mesh filename=meshes/link_01.stl; visual mesh filename=meshes/link_01.stl
- link F2_02: geometry collision mesh filename=meshes/link_02.stl; visual mesh filename=meshes/link_02.stl
- link F2_03: geometry collision mesh filename=meshes/link_03.stl; visual mesh filename=meshes/link_03.stl
- link F2_04: geometry collision mesh filename=meshes/link_04.stl; visual mesh filename=meshes/link_04.stl
- link F2_TIP: geometry collision mesh filename=meshes/link_tip_high.stl; visual mesh filename=meshes/link_tip_high.stl
- link F3_01: geometry collision mesh filename=meshes/link_01.stl; visual mesh filename=meshes/link_01.stl
- link F3_02: geometry collision mesh filename=meshes/link_02.stl; visual mesh filename=meshes/link_02.stl
- link F3_03: geometry collision mesh filename=meshes/link_03.stl; visual mesh filename=meshes/link_03.stl
- link F3_04: geometry collision mesh filename=meshes/link_04.stl; visual mesh filename=meshes/link_04.stl
- link F3_TIP: geometry collision mesh filename=meshes/link_tip_high.stl; visual mesh filename=meshes/link_tip_high.stl
- link delto_base_link: geometry collision mesh filename=meshes/delto_base_link.stl; visual mesh filename=meshes/delto_base_link.stl
