Commit message: Fixed instructions and typos

File: libs/robot_description/tesollo_DG3F/tesollo_DG3F.urdf.xacro (robot description, xacro)
@@ -418,5 +418,5 @@
             <parent link="${name_prefix}delto_base_link"/>
             <child link="${name_prefix}F3_01"/>
-            <axis xyz=".0 0.0 1.0"/>
+            <axis xyz="0.0 0.0 1.0"/>
             <limit effort="10.0" velocity="5.0" lower="-0.0872665" upper="2.00713" />
             <dynamics damping="1.1" friction="1.1"/>

Commit message: Corrected readme and urdf based on tesollo update

File: libs/robot_description/tesollo_DG3F/tesollo_DG3F.urdf.xacro (robot description, xacro)
@@ -404,5 +404,5 @@
             <parent link="${name_prefix}F2_03"/>
             <child link="${name_prefix}F2_04"/>
-            <axis xyz="0.0434 0.0 1.0"/>
+            <axis xyz="0.0 0.0 1.0"/>
             <limit effort="10.0" velocity="5.0" lower="-0.226893" upper="2.02458" />
             <dynamics damping="1.1" friction="1.1"/>
