Commit message: Got file import working

File: libs/robot_description/bimanual_arms.urdf (robot description, URDF)
Before this commit: robot bimanual_arms, 1 links, 0 joints
Links:
- link table: geometry collision mesh filename=panda/meshes/Kinect_front.stl scale=1 1 1; visual mesh filename=panda/meshes/Kinect_front.stl scale=1 1 1
