Commit message: Got panda model original model working with isaacsim...still need to modularize

File: libs/robot_description/panda/panda.urdf (robot description, URDF)
Before this commit: robot panda_kinect, 16 links, 15 joints
Links:
- link camera_body: geometry visual mesh filename=meshes/visual/kinect_model.stl

Commit message: Working on generating urdfs from xacros but need to fix relative links

File: libs/robot_description/panda/panda.urdf (robot description, URDF)
Before this commit: robot panda_kinect, 16 links, 15 joints
Links:
- removed link camera_base
- removed link camera_visor
Joints:
- removed joint camera_base_to_body
- removed joint camera_base_to_visor
- removed joint fake_base
