Commit message: Made panda into macro

File: libs/robot_description/panda/panda.urdf.xacro (robot description, xacro)
@@ -1,165 +1,163 @@
 <?xml version="1.0" encoding="utf-8"?>
-<robot name="panda" xmlns:xacro="http://www.ros.org/wiki/xacro">
-  <xacro:arg name="panda_file_prefix"  default="package://robot_description/panda"/>
-  <!-- If a parent has NOT defined panda_file_prefix as a property,
-        this sets it from the arg; otherwise the parent's property value stays. -->
-  <xacro:property name="panda_file_prefix"  value="$(arg panda_file_prefix)"/>
-  <link name="panda_link0">
-    <visual>
-      <geometry>
-        <mesh filename="${panda_file_prefix}/meshes/visual/link0.dae"/>
-      </geometry>
-    </visual>
-    <collision>
-      <geometry>
-        <mesh filename="${panda_file_prefix}/meshes/collision/link0.stl"/>
-      </geometry>
-    </collision>
-  </link>
-  <link name="panda_link1">
-    <visual>
-      <geometry>
-        <mesh filename="${panda_file_prefix}/meshes/visual/link1.dae"/>
-      </geometry>
-    </visual>
-    <collision>
-      <geometry>
-        <mesh filename="${panda_file_prefix}/meshes/collision/link1.stl"/>
-      </geometry>
-    </collision>
-  </link>
-  <joint name="panda_joint1" type="revolute">
-    <safety_controller k_position="100.0" k_velocity="40.0" soft_lower_limit="-2.8973" soft_upper_limit="2.8973"/>
-    <origin rpy="0 0 0" xyz="0 0 0.333"/>
-    <parent link="panda_link0"/>
-    <child link="panda_link1"/>
-    <axis xyz="0 0 1"/>
-    <limit effort="87" lower="-2.8973" upper="2.8973" velocity="2.1750"/>
-  </joint>
-  <link name="panda_link2">
-    <visual>
-      <geometry>
-        <mesh filename="${panda_file_prefix}/meshes/visual/link2.dae"/>
-      </geometry>
-    </visual>
-    <collision>
-      <geometry>
-        <mesh filename="${panda_file_prefix}/meshes/collision/link2.stl"/>
-      </geometry>
-    </collision>
-  </link>
-  <joint name="panda_joint2" type="revolute">
-    <safety_controller k_position="100.0" k_velocity="40.0" soft_lower_limit="-1.7628" soft_upper_limit="1.7628"/>
-    <origin rpy="-1.57079632679 0 0" xyz="0 0 0"/>
-    <parent link="panda_link1"/>
-    <child link="panda_link2"/>
-    <axis xyz="0 0 1"/>
-    <limit effort="87" lower="-1.7628" upper="1.7628" velocity="2.1750"/>
-  </joint>
-  <link name="panda_link3">
-    <visual>
-      <geometry>
-        <mesh filename="${panda_file_prefix}/meshes/visual/link3.dae"/>
-      </geometry>
-    </visual>
-    <collision>
-      <geometry>
-        <mesh filename="${panda_file_prefix}/meshes/collision/link3.stl"/>
-      </geometry>
-    </collision>
-  </link>
-  <joint name="panda_joint3" type="revolute">
-    <safety_controller k_position="100.0" k_velocity="40.0" soft_lower_limit="-2.8973" soft_upper_limit="2.8973"/>
-    <origin rpy="1.57079632679 0 0" xyz="0 -0.316 0"/>
-    <parent link="panda_link2"/>
-    <child link="panda_link3"/>
-    <axis xyz="0 0 1"/>
-    <limit effort="87" lower="-2.8973" upper="2.8973" velocity="2.1750"/>
-  </joint>
-  <link name="panda_link4">
-    <visual>
-      <geometry>
-        <mesh filename="${panda_file_prefix}/meshes/visual/link4.dae"/>
-      </geometry>
-    </visual>
-    <collision>
-      <geometry>
-        <mesh filename="${panda_file_prefix}/meshes/collision/link4.stl"/>
-      </geometry>
-    </collision>
-  </link>
-  <joint name="panda_joint4" type="revolute">
-    <safety_controller k_position="100.0" k_velocity="40.0" soft_lower_limit="-3.0718" soft_upper_limit="-0.0698"/>
-    <origin rpy="1.57079632679 0 0" xyz="0.0825 0 0"/>
-    <parent link="panda_link3"/>
-    <child link="panda_link4"/>
-    <axis xyz="0 0 1"/>
-    <limit effort="87" lower="-3.0718" upper="-0.0698" velocity="2.1750"/>
-  </joint>
-  <link name="panda_link5">
-    <visual>
-      <geometry>
-        <mesh filename="${panda_file_prefix}/meshes/visual/link5.dae"/>
-      </geometry>
-    </visual>
-    <collision>
-      <geometry>
-        <mesh filename="${panda_file_prefix}/meshes/collision/link5.stl"/>
-      </geometry>
-    </collision>
-  </link>
-  <joint name="panda_joint5" type="revolute">
-    <safety_controller k_position="100.0" k_velocity="40.0" soft_lower_limit="-2.8973" soft_upper_limit="2.8973"/>
-    <origin rpy="-1.57079632679 0 0" xyz="-0.0825 0.384 0"/>
-    <parent link="panda_link4"/>
-    <child link="panda_link5"/>
-    <axis xyz="0 0 1"/>
-    <limit effort="12" lower="-2.8973" upper="2.8973" velocity="2.6100"/>
-  </joint>
-  <link name="panda_link6">
-    <visual>
-      <geometry>
-        <mesh filename="${panda_file_prefix}/meshes/visual/link6.dae"/>
-      </geometry>
-    </visual>
-    <collision>
-      <geometry>
-        <mesh filename="${panda_file_prefix}/meshes/collision/link6.stl"/>
-      </geometry>
-    </collision>
-  </link>
-  <joint name="panda_joint6" type="revolute">
-    <safety_controller k_position="100.0" k_velocity="40.0" soft_lower_limit="-0.0175" soft_upper_limit="3.7525"/>
-    <origin rpy="1.57079632679 0 0" xyz="0 0 0"/>
-    <parent link="panda_link5"/>
-    <child link="panda_link6"/>
-    <axis xyz="0 0 1"/>
-    <limit effort="12" lower="-0.0175" upper="3.7525" velocity="2.6100"/>
-  </joint>
-  <link name="panda_link7">
-    <visual>
-      <geometry>
-        <mesh filename="${panda_file_prefix}/meshes/visual/link7.dae"/>
-      </geometry>
-    </visual>
-    <collision>
-      <geometry>
-        <mesh filename="${panda_file_prefix}/meshes/collision/link7.stl"/>
-      </geometry>
-    </collision>
-  </link>
-  <joint name="panda_joint7" type="revolute">
-    <safety_controller k_position="100.0" k_velocity="40.0" soft_lower_limit="-2.8973" soft_upper_limit="2.8973"/>
-    <origin rpy="1.57079632679 0 0" xyz="0.088 0 0"/>
-    <parent link="panda_link6"/>
-    <child link="panda_link7"/>
-    <axis xyz="0 0 1"/>
-    <limit effort="12" lower="-2.8973" upper="2.8973" velocity="2.6100"/>
-  </joint>
-  <link name="panda_link8"/>
-  <joint name="panda_joint8" type="fixed">
-    <parent link="panda_link7"/>
-    <child link="panda_link8"/>
-    <origin rpy="0 0 0" xyz="0 0 0.107"/>
-  </joint>
+<robot xmlns:xacro="http://www.ros.org/wiki/xacro">
+<xacro:macro name="panda" params="file_prefix:='package://robot_description/panda' name_prefix:=''">
+    <link name="${name_prefix}panda_link0">
+      <visual>
+        <geometry>
+          <mesh filename="${file_prefix}/meshes/visual/link0.dae"/>
+        </geometry>
+      </visual>
+      <collision>
+        <geometry>
+          <mesh filename="${file_prefix}/meshes/collision/link0.stl"/>
+        </geometry>
+      </collision>
+    </link>
+    <link name="${name_prefix}panda_link1">
+      <visual>
+        <geometry>
+          <mesh filename="${file_prefix}/meshes/visual/link1.dae"/>
+        </geometry>
+      </visual>
+      <collision>
+        <geometry>
+          <mesh filename="${file_prefix}/meshes/collision/link1.stl"/>
+        </geometry>
+      </collision>
+    </link>
+    <joint name="${name_prefix}panda_joint1" type="revolute">
+      <safety_controller k_position="100.0" k_velocity="40.0" soft_lower_limit="-2.8973" soft_upper_limit="2.8973"/>
+      <origin rpy="0 0 0" xyz="0 0 0.333"/>
+      <parent link="${name_prefix}panda_link0"/>
+      <child link="${name_prefix}panda_link1"/>
+      <axis xyz="0 0 1"/>
+      <limit effort="87" lower="-2.8973" upper="2.8973" velocity="2.1750"/>
+    </joint>
+    <link name="${name_prefix}panda_link2">
+      <visual>
+        <geometry>
+          <mesh filename="${file_prefix}/meshes/visual/link2.dae"/>
+        </geometry>
+      </visual>
+      <collision>
+        <geometry>
+          <mesh filename="${file_prefix}/meshes/collision/link2.stl"/>
+        </geometry>
+      </collision>
+    </link>
+    <joint name="${name_prefix}panda_joint2" type="revolute">
+      <safety_controller k_position="100.0" k_velocity="40.0" soft_lower_limit="-1.7628" soft_upper_limit="1.7628"/>
+      <origin rpy="-1.57079632679 0 0" xyz="0 0 0"/>
+      <parent link="${name_prefix}panda_link1"/>
+      <child link="${name_prefix}panda_link2"/>
+      <axis xyz="0 0 1"/>
+      <limit effort="87" lower="-1.7628" upper="1.7628" velocity="2.1750"/>
+    </joint>
+    <link name="${name_prefix}panda_link3">
+      <visual>
+        <geometry>
+          <mesh filename="${file_prefix}/meshes/visual/link3.dae"/>
+        </geometry>
+      </visual>
+      <collision>
+        <geometry>
+          <mesh filename="${file_prefix}/meshes/collision/link3.stl"/>
+        </geometry>
+      </collision>
+    </link>
+    <joint name="${name_prefix}panda_joint3" type="revolute">
+      <safety_controller k_position="100.0" k_velocity="40.0" soft_lower_limit="-2.8973" soft_upper_limit="2.8973"/>
+      <origin rpy="1.57079632679 0 0" xyz="0 -0.316 0"/>
+      <parent link="${name_prefix}panda_link2"/>
+      <child link="${name_prefix}panda_link3"/>
+      <axis xyz="0 0 1"/>
+      <limit effort="87" lower="-2.8973" upper="2.8973" velocity="2.1750"/>
+    </joint>
+    <link name="${name_prefix}panda_link4">
+      <visual>
+        <geometry>
+          <mesh filename="${file_prefix}/meshes/visual/link4.dae"/>
+        </geometry>
+      </visual>
+      <collision>
+        <geometry>
+          <mesh filename="${file_prefix}/meshes/collision/link4.stl"/>
+        </geometry>
+      </collision>
+    </link>
+    <joint name="${name_prefix}panda_joint4" type="revolute">
+      <safety_controller k_position="100.0" k_velocity="40.0" soft_lower_limit="-3.0718" soft_upper_limit="-0.0698"/>
+      <origin rpy="1.57079632679 0 0" xyz="0.0825 0 0"/>
+      <parent link="${name_prefix}panda_link3"/>
+      <child link="${name_prefix}panda_link4"/>
+      <axis xyz="0 0 1"/>
+      <limit effort="87" lower="-3.0718" upper="-0.0698" velocity="2.1750"/>
+    </joint>
+    <link name="${name_prefix}panda_link5">
+      <visual>
+        <geometry>
+          <mesh filename="${file_prefix}/meshes/visual/link5.dae"/>
+        </geometry>
+      </visual>
+      <collision>
+        <geometry>
+          <mesh filename="${file_prefix}/meshes/collision/link5.stl"/>
+        </geometry>
+      </collision>
+    </link>
+    <joint name="${name_prefix}panda_joint5" type="revolute">
+      <safety_controller k_position="100.0" k_velocity="40.0" soft_lower_limit="-2.8973" soft_upper_limit="2.8973"/>
+      <origin rpy="-1.57079632679 0 0" xyz="-0.0825 0.384 0"/>
+      <parent link="${name_prefix}panda_link4"/>
+      <child link="${name_prefix}panda_link5"/>
+      <axis xyz="0 0 1"/>
+      <limit effort="12" lower="-2.8973" upper="2.8973" velocity="2.6100"/>
+    </joint>
+    <link name="${name_prefix}panda_link6">
+      <visual>
+        <geometry>
+          <mesh filename="${file_prefix}/meshes/visual/link6.dae"/>
+        </geometry>
+      </visual>
+      <collision>
+        <geometry>
+          <mesh filename="${file_prefix}/meshes/collision/link6.stl"/>
+        </geometry>
+      </collision>
+    </link>
+    <joint name="${name_prefix}panda_joint6" type="revolute">
+      <safety_controller k_position="100.0" k_velocity="40.0" soft_lower_limit="-0.0175" soft_upper_limit="3.7525"/>
+      <origin rpy="1.57079632679 0 0" xyz="0 0 0"/>
+      <parent link="${name_prefix}panda_link5"/>
+      <child link="${name_prefix}panda_link6"/>
+      <axis xyz="0 0 1"/>
+      <limit effort="12" lower="-0.0175" upper="3.7525" velocity="2.6100"/>
+    </joint>
+    <link name="${name_prefix}panda_link7">
+      <visual>
+        <geometry>
+          <mesh filename="${file_prefix}/meshes/visual/link7.dae"/>
+        </geometry>
+      </visual>
+      <collision>
+        <geometry>
+          <mesh filename="${file_prefix}/meshes/collision/link7.stl"/>
+        </geometry>
+      </collision>
+    </link>
+    <joint name="${name_prefix}panda_joint7" type="revolute">
+      <safety_controller k_position="100.0" k_velocity="40.0" soft_lower_limit="-2.8973" soft_upper_limit="2.8973"/>
+      <origin rpy="1.57079632679 0 0" xyz="0.088 0 0"/>
+      <parent link="${name_prefix}panda_link6"/>
+      <child link="${name_prefix}panda_link7"/>
+      <axis xyz="0 0 1"/>
+      <limit effort="12" lower="-2.8973" upper="2.8973" velocity="2.6100"/>
+    </joint>
+    <link name="${name_prefix}panda_link8"/>
+    <joint name="${name_prefix}panda_joint8" type="fixed">
+      <parent link="${name_prefix}panda_link7"/>
+      <child link="${name_prefix}panda_link8"/>
+      <origin rpy="0 0 0" xyz="0 0 0.107"/>
+    </joint>
+  </xacro:macro>
 </robot>

File: libs/robot_description/panda/panda_hand.urdf.xacro (robot description, xacro)
@@ -1,60 +1,58 @@
 <?xml version="1.0" encoding="utf-8"?>
-<robot name="panda_hand" xmlns:xacro="http://www.ros.org/wiki/xacro">
-  <xacro:arg name="panda_file_prefix"  default="package://robot_description/panda"/>
-  <!-- If a parent has NOT defined panda_file_prefix as a property,
-        this sets it from the arg; otherwise the parent's property value stays. -->
-  <xacro:property name="panda_file_prefix"  value="$(arg panda_file_prefix)"/>
-  <link name="panda_hand">
-    <visual>
-      <geometry>
-        <mesh filename="${panda_file_prefix}/meshes/visual/hand.dae"/>
-      </geometry>
-    </visual>
-    <collision>
-      <geometry>
-        <mesh filename="${panda_file_prefix}/meshes/collision/hand.stl"/>
-      </geometry>
-    </collision>
-  </link>
-  <link name="panda_leftfinger">
-    <visual>
-      <geometry>
-        <mesh filename="${panda_file_prefix}/meshes/visual/finger.dae"/>
-      </geometry>
-    </visual>
-    <collision>
-      <geometry>
-        <mesh filename="${panda_file_prefix}/meshes/collision/finger.stl"/>
-      </geometry>
-    </collision>
-  </link>
-  <link name="panda_rightfinger">
-    <visual>
-      <origin rpy="0 0 3.14159265359" xyz="0 0 0"/>
-      <geometry>
-        <mesh filename="${panda_file_prefix}/meshes/visual/finger.dae"/>
-      </geometry>
-    </visual>
-    <collision>
-      <origin rpy="0 0 3.14159265359" xyz="0 0 0"/>
-      <geometry>
-        <mesh filename="${panda_file_prefix}/meshes/collision/finger.stl"/>
-      </geometry>
-    </collision>
-  </link>
-  <joint name="panda_finger_joint1" type="prismatic">
-    <parent link="panda_hand"/>
-    <child link="panda_leftfinger"/>
-    <origin rpy="0 0 0" xyz="0 0 0.0584"/>
-    <axis xyz="0 1 0"/>
-    <limit effort="20" lower="0.0" upper="0.04" velocity="0.2"/>
-  </joint>
-  <joint name="panda_finger_joint2" type="prismatic">
-    <parent link="panda_hand"/>
-    <child link="panda_rightfinger"/>
-    <origin rpy="0 0 0" xyz="0 0 0.0584"/>
-    <axis xyz="0 -1 0"/>
-    <limit effort="20" lower="0.0" upper="0.04" velocity="0.2"/>
-    <mimic joint="panda_finger_joint1"/>
-  </joint>
+<robot xmlns:xacro="http://www.ros.org/wiki/xacro">
+  <xacro:macro name="panda_hand" params="file_prefix:='package://robot_description/panda' name_prefix:=''">
+    <link name="${name_prefix}panda_hand">
+      <visual>
+        <geometry>
+          <mesh filename="${file_prefix}/meshes/visual/hand.dae"/>
+        </geometry>
+      </visual>
+      <collision>
+        <geometry>
+          <mesh filename="${file_prefix}/meshes/collision/hand.stl"/>
+        </geometry>
+      </collision>
+    </link>
+    <link name="${name_prefix}panda_leftfinger">
+      <visual>
+        <geometry>
+          <mesh filename="${file_prefix}/meshes/visual/finger.dae"/>
+        </geometry>
+      </visual>
+      <collision>
+        <geometry>
+          <mesh filename="${file_prefix}/meshes/collision/finger.stl"/>
+        </geometry>
+      </collision>
+    </link>
+    <link name="${name_prefix}panda_rightfinger">
+      <visual>
+        <origin rpy="0 0 3.14159265359" xyz="0 0 0"/>
+        <geometry>
+          <mesh filename="${file_prefix}/meshes/visual/finger.dae"/>
+        </geometry>
+      </visual>
+      <collision>
+        <origin rpy="0 0 3.14159265359" xyz="0 0 0"/>
+        <geometry>
+          <mesh filename="${file_prefix}/meshes/collision/finger.stl"/>
+        </geometry>
+      </collision>
+    </link>
+    <joint name="${name_prefix}panda_finger_joint1" type="prismatic">
+      <parent link="${name_prefix}panda_hand"/>
+      <child link="${name_prefix}panda_leftfinger"/>
+      <origin rpy="0 0 0" xyz="0 0 0.0584"/>
+      <axis xyz="0 1 0"/>
+      <limit effort="20" lower="0.0" upper="0.04" velocity="0.2"/>
+    </joint>
+    <joint name="${name_prefix}panda_finger_joint2" type="prismatic">
+      <parent link="${name_prefix}panda_hand"/>
+      <child link="${name_prefix}panda_rightfinger"/>
+      <origin rpy="0 0 0" xyz="0 0 0.0584"/>
+      <axis xyz="0 -1 0"/>
+      <limit effort="20" lower="0.0" upper="0.04" velocity="0.2"/>
+      <mimic joint="${name_prefix}panda_finger_joint1"/>
+    </joint>
+    </xacro:macro>
 </robot>

File: libs/robot_description/panda/panda_w_hand.urdf.xacro (robot description, xacro)
@@ -1,13 +1,15 @@
 <?xml version="1.0" encoding="utf-8"?>
 <robot  name="panda_w_hand" xmlns:xacro="http://www.ros.org/wiki/xacro">
-  <xacro:arg name="panda_file_prefix"  default="package://robot_description/panda"/>
-  <!-- Args for included files -->
-  <xacro:property name="panda_file_prefix"  value="$(arg panda_file_prefix)"/>
-  <xacro:include filename="${panda_file_prefix}/panda_hand.urdf.xacro" />
-  <xacro:include filename="${panda_file_prefix}/panda.urdf.xacro" />
+  <xacro:arg name="file_prefix"  default="package://robot_description/panda"/>
+  <xacro:arg name="name_prefix"  default=""/>
+  <!-- Macros -->
+  <xacro:include filename="$(arg file_prefix)/panda_hand.urdf.xacro"/>
+  <xacro:include filename="$(arg file_prefix)/panda.urdf.xacro"/>
+  <xacro:panda_hand name_prefix="$(arg name_prefix)" file_prefix="$(arg file_prefix)"/>
+  <xacro:panda name_prefix="$(arg name_prefix)" file_prefix="$(arg file_prefix)"/>
   <!-- Connection Joints -->
-  <joint name="panda_hand_joint" type="fixed">
-    <parent link="panda_link8"/>
-    <child link="panda_hand"/>
+  <joint name="$(arg name_prefix)panda_hand_joint" type="fixed">
+    <parent link="$(arg name_prefix)panda_link8"/>
+    <child link="$(arg name_prefix)panda_hand"/>
     <origin rpy="0 0 0" xyz="0 0 0"/>
   </joint>

Commit message: Added mass to pandas

File: libs/robot_description/panda/panda.urdf.xacro (robot description, xacro)
@@ -13,4 +13,9 @@
         </geometry>
       </collision>
+      <inertial>
+        <origin xyz="-0.0172 0.0004 0.0745" rpy="0 0 0"/>
+        <mass value="2.3966"/>
+        <inertia ixx="0.0090" ixy="0.0000" ixz="0.0020" iyy="0.0115" iyz="0.0000" izz="0.0085"/>
+      </inertial>
     </link>
     <link name="${name_prefix}panda_link1">
@@ -25,4 +30,10 @@
         </geometry>
       </collision>
+      <inertial>
+        <origin xyz="0.00033 -0.02204 -0.04762" rpy="0 0 0"/>
+        <mass value="2.7907"/>
+        <inertia ixx="0.01564782655" ixy="0.00000531236" ixz="-0.00003676721"
+                iyy="0.01439883526" iyz="-0.00248480843" izz="0.00500443991"/>
+      </inertial>
     </link>
     <joint name="${name_prefix}panda_joint1" type="revolute">
@@ -45,4 +56,10 @@
         </geometry>
       </collision>
+      <inertial>
+        <origin xyz="0.00038 -0.09211 0.01908" rpy="0 0 0"/>
+        <mass value="2.5420"/>
+        <inertia ixx="0.01662427728" ixy="0.00003086077" ixz="0.00000835940"
+                iyy="0.00462501261" iyz="0.00355899830" izz="0.01545124526"/>
+      </inertial>
     </link>
     <joint name="${name_prefix}panda_joint2" type="revolute">
@@ -65,4 +82,10 @@
         </geometry>
       </collision>
+      <inertial>
+        <origin xyz="0.05152 0.01696 -0.02971" rpy="0 0 0"/>
+        <mass value="2.2513"/>
+        <inertia ixx="0.00631741992" ixy="0.00097309955" ixz="0.00292525834"
+                iyy="0.00866285493" iyz="0.00093469224" izz="0.00657804051"/>
+      </inertial>
     </link>
     <joint name="${name_prefix}panda_joint3" type="revolute">
@@ -85,4 +108,10 @@
         </geometry>
       </collision>
+      <inertial>
+        <origin xyz="-0.05113 0.05825 0.01698" rpy="0 0 0"/>
+        <mass value="2.2037"/>
+        <inertia ixx="0.00784585566" ixy="-0.00339591957" ixz="0.00158704074"
+                iyy="0.00649543136" iyz="-0.00181477884" izz="0.01003079917"/>
+      </inertial>
     </link>
     <joint name="${name_prefix}panda_joint4" type="revolute">
@@ -105,4 +134,10 @@
         </geometry>
       </collision>
+      <inertial>
+        <origin xyz="-0.00005 0.03730 -0.09280" rpy="0 0 0"/>
+        <mass value="2.2855"/>
+        <inertia ixx="0.02297014781" ixy="-0.00000949345" ixz="-0.00002063156"
+                iyy="0.02095060919" iyz="0.00382345782" izz="0.00430606551"/>
+      </inertial>
     </link>
     <joint name="${name_prefix}panda_joint5" type="revolute">
@@ -125,4 +160,10 @@
         </geometry>
       </collision>
+      <inertial>
+        <origin xyz="0.06572 -0.00371 0.00153" rpy="0 0 0"/>
+        <mass value="1.353"/>
+        <inertia ixx="0.00087964522" ixy="-0.00021487814" ixz="-0.00011911662"
+                iyy="0.00277796968" iyz="0.00001274322" izz="0.00286701969"/>
+      </inertial>
     </link>
     <joint name="${name_prefix}panda_joint6" type="revolute">
@@ -145,4 +186,10 @@
         </geometry>
       </collision>
+      <inertial>
+        <origin xyz="0.00089 -0.00044 0.05491" rpy="0 0 0"/>
+        <mass value="0.35973"/>
+        <inertia ixx="0.00019541063" ixy="0.00000165231" ixz="0.00000148826"
+                iyy="0.00019210361" iyz="-0.00000131132" izz="0.00017936256"/>
+      </inertial>
     </link>
     <joint name="${name_prefix}panda_joint7" type="revolute">

File: libs/robot_description/panda/panda_hand.urdf.xacro (robot description, xacro)
@@ -13,4 +13,10 @@
         </geometry>
       </collision>
+      <inertial>
+        <origin xyz="-0.0000376 0.0119128 0.0207260" rpy="0 0 0"/>
+        <mass value="0.6544"/>
+        <inertia ixx="0.00186" ixy="0.00000" ixz="0.00000"
+                 iyy="0.00030" iyz="-0.00002" izz="0.00174"/>
+      </inertial>
     </link>
     <link name="${name_prefix}panda_leftfinger">
@@ -25,4 +31,10 @@
         </geometry>
       </collision>
+      <inertial>
+        <origin xyz="0 0.0152850 0.0219675" rpy="0 0 0"/>
+        <mass value="0.0291"/>
+        <inertia ixx="0.00000849" ixy="0.00000000" ixz="0.00000000"
+                 iyy="0.00000853" iyz="-0.00000106" izz="0.00000177"/>
+      </inertial>
     </link>
     <link name="${name_prefix}panda_rightfinger">
@@ -39,4 +51,10 @@
         </geometry>
       </collision>
+      <inertial>
+        <origin xyz="0 0.0152850 0.0219675" rpy="0 0 0"/>
+        <mass value="0.0291"/>
+        <inertia ixx="0.00000849" ixy="0.00000000" ixz="0.00000000"
+                 iyy="0.00000853" iyz="-0.00000106" izz="0.00000177"/>
+      </inertial>
     </link>
     <joint name="${name_prefix}panda_finger_joint1" type="prismatic">
@@ -55,4 +73,4 @@
       <mimic joint="${name_prefix}panda_finger_joint1"/>
     </joint>
-    </xacro:macro>
+  </xacro:macro>
 </robot>
