Commit message: Turned kinect and ft sensor into macros and updated readme

File: libs/robot_description/ft_sensor/ft_sensor.urdf.xacro (robot description, xacro)
@@ -1,20 +1,18 @@
 <?xml version="1.0" encoding="utf-8"?>
 <!-- Force Torque Sensor -->
-<robot name="ft_sensor" xmlns:xacro="http://www.ros.org/wiki/xacro">
-  <xacro:arg name="ft_sensor_file_prefix"  default="package://robot_description/ft_sensor"/>
-  <!-- If a parent has NOT defined ft_sensor_file_prefix as a property,
-        this sets it from the arg; otherwise the parent's property value stays. -->
-  <xacro:property name="ft_sensor_file_prefix"  value="$(arg ft_sensor_file_prefix)"/>
-  <link name="ft_sensor_link">
-    <visual>
-      <geometry>
-        <mesh filename="${ft_sensor_file_prefix}/meshes/force_torque_sensor.dae"/>
-      </geometry>
-    </visual>
-    <collision>
-      <geometry>
-        <mesh filename="${ft_sensor_file_prefix}/meshes/force_torque_sensor.stl"/>
-      </geometry>
-    </collision>
-  </link>
+<robot xmlns:xacro="http://www.ros.org/wiki/xacro">
+  <xacro:macro name="ft_sensor" params="file_prefix:='package://robot_description/ft_sensor' name_prefix:='' ">
+    <link name="${name_prefix}ft_sensor_link">
+      <visual>
+        <geometry>
+          <mesh filename="${file_prefix}/meshes/force_torque_sensor.dae"/>
+        </geometry>
+      </visual>
+      <collision>
+        <geometry>
+          <mesh filename="${file_prefix}/meshes/force_torque_sensor.stl"/>
+        </geometry>
+      </collision>
+    </link>
+  </xacro:macro>
 </robot>

File: libs/robot_description/kinect/kinect.urdf.xacro (robot description, xacro)
@@ -1,30 +1,28 @@
 <?xml version="1.0" encoding="utf-8"?>
-<robot name="kinect" xmlns:xacro="http://www.ros.org/wiki/xacro">
-  <xacro:arg name="kinect_file_prefix"  default="package://robot_description/kinect"/>
-  <!-- If a parent has NOT defined kinect_file_prefix as a property,
-        this sets it from the arg; otherwise the parent's property value stays. -->
-  <xacro:property name="kinect_file_prefix"  value="$(arg kinect_file_prefix)"/>
-  <link name="camera_body">
-    <visual>
-      <origin rpy="0 3.1416 0"  xyz=".047 0.04 0.0115"/>
-      <geometry>
-        <mesh filename="${kinect_file_prefix}/meshes/kinect.stl"/>
-      </geometry>
-      <material name="white"/>
-    </visual>
-  </link>
-  <link name="camera_base">
-  </link>
-  <link name="camera_visor">
-  </link>
-  <joint name="camera_base_to_body" type="fixed">
-    <parent link="camera_base"/>
-    <child link="camera_body"/>
-    <origin rpy="0. 0. 0." xyz="-0.0757 0. 0.008"/>
-  </joint>
-  <joint name="camera_base_to_visor" type="fixed">
-    <parent link="camera_base"/>
-    <child link="camera_visor"/>
-    <origin rpy="0. 0. 0." xyz="0. 0. 0."/>
-  </joint>
+<robot xmlns:xacro="http://www.ros.org/wiki/xacro">
+  <xacro:macro name="kinect" params="file_prefix:='package://robot_description/kinect' name_prefix:='' ">
+    <link name="${name_prefix}camera_body">
+      <visual>
+        <origin rpy="0 3.1416 0"  xyz=".047 0.04 0.0115"/>
+        <geometry>
+          <mesh filename="${file_prefix}/meshes/kinect.stl"/>
+        </geometry>
+        <material name="white"/>
+      </visual>
+    </link>
+    <link name="${name_prefix}camera_base">
+    </link>
+    <link name="${name_prefix}camera_visor">
+    </link>
+    <joint name="${name_prefix}camera_base_to_body" type="fixed">
+      <parent link="${name_prefix}camera_base"/>
+      <child link="${name_prefix}camera_body"/>
+      <origin rpy="0. 0. 0." xyz="-0.0757 0. 0.008"/>
+    </joint>
+    <joint name="${name_prefix}camera_base_to_visor" type="fixed">
+      <parent link="${name_prefix}camera_base"/>
+      <child link="${name_prefix}camera_visor"/>
+      <origin rpy="0. 0. 0." xyz="0. 0. 0."/>
+    </joint>
+  </xacro:macro>
 </robot>
