Commit message: Added all objects to bimanual system, now need to align them properly.

File: libs/robot_description/composites/bimanual_arms.urdf.xacro (robot description, xacro)
@@ -1,26 +1,40 @@
-<robot name="bimanual_arms">
+<?xml version="1.0" encoding="utf-8"?>
+<robot  name="bimanual_arms" xmlns:xacro="http://www.ros.org/wiki/xacro">
+  <xacro:arg name="composite_file_prefix"  default="package://robot_description/composites"/>
+  <xacro:arg name="panda_file_prefix"  default="package://robot_description/panda"/>
+  <xacro:arg name="tesollo_DG3F_file_prefix"  default="package://robot_description/tesollo"/>
+  <xacro:include filename="$(arg composite_file_prefix)/panda_w_tesollo.urdf.xacro"/>
+  <xacro:panda_w_tesollo name_prefix="left_" panda_file_prefix="$(arg panda_file_prefix)"
+                 tesollo_DG3F_file_prefix="$(arg tesollo_DG3F_file_prefix)"/>
+  <xacro:panda_w_tesollo name_prefix="right_" panda_file_prefix="$(arg panda_file_prefix)"
+                 tesollo_DG3F_file_prefix="$(arg tesollo_DG3F_file_prefix)"/>
+  <!-- Connection Joints -->
+  <joint name="left_panda_mount" type="fixed">
+    <parent link="table"/>
+    <child link="left_panda_link0"/>
+    <origin rpy="0 0 0" xyz="0 -1 0"/>
+  </joint>
+  <joint name="right_panda_mount" type="fixed">
+    <parent link="table"/>
+    <child link="right_panda_link0"/>
+    <origin rpy="0 0 0" xyz="0 1 0"/>
+  </joint>
+  <!-- TABLE -->
   <link name="table">
-    <inertial>
+    <visual>
       <origin xyz="0 0 0" rpy="0 0 0"/>
-      <mass value="1.0"/> <!-- in kilograms -->
-      <inertia ixx="0.001" ixy="0.0" ixz="0.0"
-               iyy="0.001" iyz="0.0"
-               izz="0.001"/>
-    </inertial>
+      <geometry>
+        <box size="1.2 0.8 0.04"/>
+      </geometry>
+      <material name="wood">
+        <color rgba="0.70 0.50 0.30 1.0"/>
+      </material>
+    </visual>
     <collision>
       <origin xyz="0 0 0" rpy="0 0 0"/>
       <geometry>
-        <mesh filename="panda/meshes/Kinect_front.stl" scale="1 1 1"/>
+        <box size="1.2 0.8 0.04"/>
       </geometry>
     </collision>
-    <visual>
-      <origin xyz="0 0 0" rpy="0 0 0"/>
-      <geometry>
-        <mesh filename="panda/meshes/Kinect_front.stl" scale="1 1 1"/>
-      </geometry>
-      <material name="blue">
-        <color rgba="0 0 1 1"/>
-      </material>
-    </visual>
   </link>
 </robot>

File: libs/robot_description/composites/panda_w_tesollo.urdf.xacro (robot description, xacro)
@@ -1,18 +1,33 @@
 <?xml version="1.0" encoding="utf-8"?>
 <robot  name="panda_w_tesollo" xmlns:xacro="http://www.ros.org/wiki/xacro">
+  <xacro:arg name="standalone" default="false"/>
   <xacro:arg name="panda_file_prefix"  default="package://robot_description/panda"/>
   <xacro:arg name="tesollo_DG3F_file_prefix"  default="package://robot_description/tesollo"/>
   <xacro:arg name="name_prefix"  default=""/>
-  <!-- Macros -->
   <xacro:include filename="$(arg panda_file_prefix)/panda.urdf.xacro"/>
   <xacro:include filename="$(arg tesollo_DG3F_file_prefix)/tesollo_DG3F.urdf.xacro"/>
-  <xacro:panda name_prefix="$(arg name_prefix)" file_prefix="$(arg panda_file_prefix)"/>
-  <xacro:tesollo_DG3F name_prefix="$(arg name_prefix)" file_prefix="$(arg tesollo_DG3F_file_prefix)"/>
-  <!-- Connection Joints -->
-  <!-- TODO: Check rotation and height -->
-  <joint name="$(arg name_prefix)panda_gripper_joint" type="fixed">
-    <parent link="$(arg name_prefix)panda_link8"/>
-    <child link="$(arg name_prefix)delto_base_link"/>
-    <origin rpy="0 0 0" xyz="0 0 0.106"/>
-  </joint>
+  <xacro:macro name="panda_w_tesollo"
+               params="
+                 name_prefix:=''
+                 panda_file_prefix:='package://robot_description/panda'
+                 tesollo_DG3F_file_prefix:='package://robot_description/tesollo'">
+    <xacro:panda name_prefix="${name_prefix}" file_prefix="${panda_file_prefix}"/>
+    <xacro:tesollo_DG3F name_prefix="${name_prefix}" file_prefix="${tesollo_DG3F_file_prefix}"/>
+    <!-- Connection Joints -->
+    <!-- TODO: Check rotation and height -->
+    <joint name="${name_prefix}panda_gripper_joint" type="fixed">
+      <parent link="${name_prefix}panda_link8"/>
+      <child link="${name_prefix}delto_base_link"/>
+      <origin rpy="0 0 0" xyz="0 0 0.106"/>
+    </joint>
+  </xacro:macro>
+  <!-- ===== Standalone launcher =====
+      Only emits a <robot> when standalone:=true (default)
+      When included in another robot, set standalone:=false -->
+  <xacro:if value="$(arg standalone)">
+    <xacro:panda_w_tesollo
+      name_prefix="$(arg name_prefix)"
+      panda_file_prefix="$(arg panda_file_prefix)"
+      tesollo_DG3F_file_prefix="$(arg tesollo_DG3F_file_prefix)"/>
+  </xacro:if>
 </robot>

File: libs/robot_description/tesollo_DG3F/tesollo_DG3F.urdf.xacro (robot description, xacro)
@@ -11,11 +11,8 @@
 <robot xmlns:xacro="http://www.ros.org/wiki/xacro">
    <xacro:macro name="tesollo_DG3F" params="file_prefix:='package://robot_description/tesollo_DG3F' name_prefix:='' ">
-        <material name="silver">
-            <color rgba="0.700 0.700 0.700 1.000"/>
-        </material>
-        <material name="black">
+        <material name="${name_prefix}black">
             <color rgba="0.196 0.196 0.196 1.0"/>
         </material>
-        <material name="white">
+        <material name="${name_prefix}white">
             <color rgba="1.0 1.0 1.0 1.0"/>
         </material>
@@ -31,5 +28,5 @@
                 <mesh filename="${file_prefix}/meshes/delto_base_link.stl"/>
                 </geometry>
-                <material name="black"/>
+                <material name="${name_prefix}black"/>
             </visual>
             <collision>
@@ -51,5 +48,5 @@
                 <mesh filename="${file_prefix}/meshes/link_01.stl"/>
                 </geometry>
-                <material name="black"/>
+                <material name="${name_prefix}black"/>
             </visual>
             <collision>
@@ -71,5 +68,5 @@
                 <mesh filename="${file_prefix}/meshes/link_02.stl"/>
                 </geometry>
-                <material name="black"/>
+                <material name="${name_prefix}black"/>
             </visual>
             <collision>
@@ -91,5 +88,5 @@
                 <mesh filename="${file_prefix}/meshes/link_03.stl"/>
                 </geometry>
-                <material name="black"/>
+                <material name="${name_prefix}black"/>
             </visual>
             <collision>
@@ -111,5 +108,5 @@
                 <mesh filename="${file_prefix}/meshes/link_04.stl"/>
                 </geometry>
-                <material name="black"/>
+                <material name="${name_prefix}black"/>
             </visual>
             <collision>
@@ -131,5 +128,5 @@
                 <mesh filename="${file_prefix}/meshes/link_tip_high.stl"/>
                 </geometry>
-                <material name="white"/>
+                <material name="${name_prefix}white"/>
             </visual>
             <collision>
@@ -151,5 +148,5 @@
                 <mesh filename="${file_prefix}/meshes/link_01.stl"/>
                 </geometry>
-                <material name="black"/>
+                <material name="${name_prefix}black"/>
             </visual>
             <collision>
@@ -171,5 +168,5 @@
                 <mesh filename="${file_prefix}/meshes/link_02.stl"/>
                 </geometry>
-                <material name="black"/>
+                <material name="${name_prefix}black"/>
             </visual>
             <collision>
@@ -191,5 +188,5 @@
                 <mesh filename="${file_prefix}/meshes/link_03.stl"/>
                 </geometry>
-                <material name="black"/>
+                <material name="${name_prefix}black"/>
             </visual>
             <collision>
@@ -211,5 +208,5 @@
                 <mesh filename="${file_prefix}/meshes/link_04.stl"/>
                 </geometry>
-                <material name="black"/>
+                <material name="${name_prefix}black"/>
             </visual>
             <collision>
@@ -231,5 +228,5 @@
                 <mesh filename="${file_prefix}/meshes/link_tip_high.stl"/>
                 </geometry>
-                <material name="white"/>
+                <material name="${name_prefix}white"/>
             </visual>
             <collision>
@@ -251,5 +248,5 @@
                 <mesh filename="${file_prefix}/meshes/link_01.stl"/>
                 </geometry>
-                <material name="black"/>
+                <material name="${name_prefix}black"/>
             </visual>
             <collision>
@@ -271,5 +268,5 @@
                 <mesh filename="${file_prefix}/meshes/link_02.stl"/>
                 </geometry>
-                <material name="black"/>
+                <material name="${name_prefix}black"/>
             </visual>
             <collision>
@@ -291,5 +288,5 @@
                 <mesh filename="${file_prefix}/meshes/link_03.stl"/>
                 </geometry>
-                <material name="black"/>
+                <material name="${name_prefix}black"/>
             </visual>
             <collision>
@@ -311,5 +308,5 @@
                 <mesh filename="${file_prefix}/meshes/link_04.stl"/>
                 </geometry>
-                <material name="black"/>
+                <material name="${name_prefix}black"/>
             </visual>
             <collision>
@@ -331,5 +328,5 @@
                 <mesh filename="${file_prefix}/meshes/link_tip_high.stl"/>
                 </geometry>
-                <material name="white"/>
+                <material name="${name_prefix}white"/>
             </visual>
             <collision>

Commit message: Measured bimanual setup

File: libs/robot_description/composites/bimanual_arms.urdf.xacro (robot description, xacro)
@@ -13,10 +13,10 @@
     <parent link="table"/>
     <child link="left_panda_link0"/>
-    <origin rpy="0 0 0" xyz="0 -1 0"/>
+    <origin rpy="0 0 0" xyz="-0.558 -0.092 0.0225"/>
   </joint>
   <joint name="right_panda_mount" type="fixed">
     <parent link="table"/>
     <child link="right_panda_link0"/>
-    <origin rpy="0 0 0" xyz="0 1 0"/>
+    <origin rpy="0 0 3.14" xyz="0.5588 -0.092 0.0225"/>
   </joint>
   <!-- TABLE -->
@@ -25,5 +25,5 @@
       <origin xyz="0 0 0" rpy="0 0 0"/>
       <geometry>
-        <box size="1.2 0.8 0.04"/>
+        <box size="1.8288 0.62865 0.045"/>
       </geometry>
       <material name="wood">
@@ -34,5 +34,5 @@
       <origin xyz="0 0 0" rpy="0 0 0"/>
       <geometry>
-        <box size="1.2 0.8 0.04"/>
+        <box size="1.8288 0.62865 0.045"/>
       </geometry>
     </collision>

Commit message: Fixed table height

File: libs/robot_description/composites/bimanual_arms.urdf.xacro (robot description, xacro)
@@ -11,15 +11,16 @@
   <!-- Connection Joints -->
   <joint name="left_panda_mount" type="fixed">
-    <parent link="table"/>
+    <parent link="table_top"/>
     <child link="left_panda_link0"/>
     <origin rpy="0 0 0" xyz="-0.558 -0.092 0.0225"/>
   </joint>
   <joint name="right_panda_mount" type="fixed">
-    <parent link="table"/>
+    <parent link="table_top"/>
     <child link="right_panda_link0"/>
     <origin rpy="0 0 3.14" xyz="0.5588 -0.092 0.0225"/>
   </joint>
   <!-- TABLE -->
-  <link name="table">
+  <link name="table"/>
+  <link name="table_top">
     <visual>
       <origin xyz="0 0 0" rpy="0 0 0"/>
@@ -38,3 +39,8 @@
     </collision>
   </link>
+  <joint name="table_top_link" type="fixed">
+    <parent link="table"/>
+    <child link="table_top"/>
+    <origin xyz="0 0 0.9144" rpy="0 0 0"/>
+  </joint>
 </robot>
