Commit message: Made tesollo into macro

File: libs/robot_description/composites/panda_w_tesollo.urdf.xacro (robot description, xacro)
@@ -3,14 +3,15 @@
   <xacro:arg name="panda_file_prefix"  default="package://robot_description/panda"/>
   <xacro:arg name="tesollo_DG3F_file_prefix"  default="package://robot_description/tesollo"/>
-  <!-- Args for included files -->
-  <xacro:property name="panda_file_prefix"  value="$(arg panda_file_prefix)"/>
-  <xacro:property name="tesollo_DG3F_file_prefix"  value="$(arg tesollo_DG3F_file_prefix)"/>
-  <xacro:include filename="${panda_file_prefix}/panda.urdf.xacro" />
-  <xacro:include filename="${tesollo_DG3F_file_prefix}/tesollo_DG3F.urdf.xacro" />
+  <xacro:arg name="name_prefix"  default=""/>
+  <!-- Macros -->
+  <xacro:include filename="$(arg panda_file_prefix)/panda.urdf.xacro"/>
+  <xacro:include filename="$(arg tesollo_DG3F_file_prefix)/tesollo_DG3F.urdf.xacro"/>
+  <xacro:panda name_prefix="$(arg name_prefix)" file_prefix="$(arg panda_file_prefix)"/>
+  <xacro:tesollo_DG3F name_prefix="$(arg name_prefix)" file_prefix="$(arg tesollo_DG3F_file_prefix)"/>
   <!-- Connection Joints -->
   <!-- TODO: Check rotation and height -->
-  <joint name="panda_gripper_joint" type="fixed">
-    <parent link="panda_link8"/>
-    <child link="delto_base_link"/>
+  <joint name="$(arg name_prefix)panda_gripper_joint" type="fixed">
+    <parent link="$(arg name_prefix)panda_link8"/>
+    <child link="$(arg name_prefix)delto_base_link"/>
     <origin rpy="0 0 0" xyz="0 0 0.106"/>
   </joint>

File: libs/robot_description/panda/panda.urdf.xacro (robot description, xacro)
@@ -1,5 +1,5 @@
 <?xml version="1.0" encoding="utf-8"?>
 <robot xmlns:xacro="http://www.ros.org/wiki/xacro">
-<xacro:macro name="panda" params="file_prefix:='package://robot_description/panda' name_prefix:=''">
+  <xacro:macro name="panda" params="file_prefix:='package://robot_description/panda' name_prefix:=''">
     <link name="${name_prefix}panda_link0">
       <visual>

File: libs/robot_description/tesollo_DG3F/tesollo_DG3F.urdf.xacro (robot description, xacro)
@@ -9,451 +9,449 @@
    * https://tesollo.com/dg-3f/
 -->
-<robot name="tesollo_DG3F"  xmlns:xacro="http://www.ros.org/wiki/xacro">
-  <xacro:arg name="tesollo_DG3F_file_prefix"  default="package://robot_description/tesollo_DG3F"/>
-  <!-- If a parent has NOT defined ft_sensor_file_prefix as a property,
-        this sets it from the arg; otherwise the parent's property value stays. -->
-  <xacro:property name="tesollo_DG3F_file_prefix"  value="$(arg tesollo_DG3F_file_prefix)"/>
-   <material name="silver">
-      <color rgba="0.700 0.700 0.700 1.000"/>
-   </material>
-   <material name="black">
-      <color rgba="0.196 0.196 0.196 1.0"/>
-   </material>
-   <material name="white">
-      <color rgba="1.0 1.0 1.0 1.0"/>
-   </material>
-   <link name="delto_base_link">
-      <inertial>
-         <origin xyz="0.00045499721796859983 -2.051648304165415e-06 -0.05218562175888181" rpy="5.671320207730568e-06 0.0032948722942074404 -0.00044870150924543735"/>
-         <mass value="0.370"/>
-         <inertia ixx="0.0009935903471030175" iyy="0.000980251548061173" izz="0.0003178199035240808" ixy="0" ixz="0" iyz="0"/>
-      </inertial>
-      <visual>
-         <origin xyz="0.00045499721796859983 -2.051648304165415e-06 -0.05218562175888181" rpy="5.671320207730568e-06 0.0032948722942074404 -0.00044870150924543735"/>
-         <geometry>
-            <mesh filename="${tesollo_DG3F_file_prefix}/meshes/delto_base_link.stl"/>
-         </geometry>
-         <material name="black"/>
-      </visual>
-      <collision>
-         <origin xyz="0.00045499721796859983 -2.051648304165415e-06 -0.05218562175888181" rpy="5.671320207730568e-06 0.0032948722942074404 -0.00044870150924543735"/>
-         <geometry>
-            <mesh filename="${tesollo_DG3F_file_prefix}/meshes/delto_base_link.stl"/>
-         </geometry>
-      </collision>
-   </link>
-   <link name="F1_01">
-      <inertial>
-         <origin xyz="0.0003906 3.121e-08 -0.014" rpy= "-0.17662368646091148 -1.9303231388878572e-06 1.5707855116626381"/>
-         <mass value="0.061"/>
-         <inertia ixx="1.924000000025899e-05" iyy="1.709411627342488e-05" izz="5.9478837263161295e-06" ixy="0" ixz="0" iyz="0"/>
-      </inertial>
-      <visual>
-         <origin xyz="0.0018977016221143523 -1.0017682763976983e-06 -0.022983822146236326" rpy="-0.1443920950720977 1.9855029389503898e-05 1.5709191233325221"/>
-         <geometry>
-            <mesh filename="${tesollo_DG3F_file_prefix}/meshes/link_01.stl"/>
-         </geometry>
-         <material name="black"/>
-      </visual>
-      <collision>
-         <origin xyz="0.0018977016221143523 -1.0017682763976983e-06 -0.022983822146236326" rpy="-0.1443920950720977 1.9855029389503898e-05 1.5709191233325221"/>
-         <geometry>
-            <mesh filename="${tesollo_DG3F_file_prefix}/meshes/link_01.stl"/>
-         </geometry>
-      </collision>
-   </link>
-   <link name="F1_02">
-      <inertial>
-         <origin xyz="0.01 3.444e-06 0.016" rpy="-0.0036890516412144943 0.31688564121750695 -0.0027736178951144786"/>
-         <mass value="0.025"/>
-         <inertia ixx="7.164797732610912e-06" iyy="6.31301833122199e-06" izz="3.274183936167101e-06" ixy="0" ixz="0" iyz="0"/>
-      </inertial>
-      <visual>
-         <origin xyz="0.010322007813576017 0.000267674195662055 0.013590600703218703" rpy="-0.03118104794815292 0.3757385725887219 -0.024334342208719002"/>
-         <geometry>
-            <mesh filename="${tesollo_DG3F_file_prefix}/meshes/link_02.stl"/>
-         </geometry>
-         <material name="black"/>
-      </visual>
-      <collision>
-         <origin xyz="0.010322007813576017 0.000267674195662055 0.013590600703218703" rpy="-0.03118104794815292 0.3757385725887219 -0.024334342208719002"/>
-         <geometry>
-            <mesh filename="${tesollo_DG3F_file_prefix}/meshes/link_02.stl"/>
-         </geometry>
-      </collision>
-   </link>
-   <link name="F1_03">
-      <inertial>
-         <origin xyz="0.014 -0.0004527 -3.953e-05" rpy="1.5651066808062148 -0.0008576993469346927 1.5562600280492769"/>
-         <mass value="0.051"/>
-         <inertia ixx="1.6912201686125405e-05" iyy="1.4940271596370447e-05" izz="6.505526717504149e-06" ixy="0" ixz="0" iyz="0"/>
-      </inertial>
-      <visual>
-         <origin xyz="0.019034639558839914 -0.0007611783816217545 0.00015734818842133856" rpy="1.5405533073968862 -0.0023628127138719535 1.5994547590929262"/>
-         <geometry>
-            <mesh filename="${tesollo_DG3F_file_prefix}/meshes/link_03.stl"/>
-         </geometry>
-         <material name="black"/>
-      </visual>
-      <collision>
-         <origin xyz="0.019034639558839914 -0.0007611783816217545 0.00015734818842133856" rpy="1.5405533073968862 -0.0023628127138719535 1.5994547590929262"/>
-         <geometry>
-            <mesh filename="${tesollo_DG3F_file_prefix}/meshes/link_03.stl"/>
-         </geometry>
-      </collision>
-   </link>
-   <link name="F1_04">
-      <inertial>
-         <origin xyz="0.012 -0.0002269 -4.676e-05" rpy="1.5668480451228681 -0.0008686188531681349 1.5829731507939977"/>
-         <mass value="0.058"/>
-         <inertia ixx="1.0860820276783573e-05" iyy="9.902070548178027e-06" izz="5.330109175038405e-06" ixy="0" ixz="0" iyz="0"/>
-      </inertial>
-      <visual>
-         <origin xyz="0.011992289866897352 -0.0007726988011287212 -5.201111709052532e-06" rpy="1.5745317514920234 0.003601150001683928 1.6650413701206925"/>
-         <geometry>
-            <mesh filename="${tesollo_DG3F_file_prefix}/meshes/link_04.stl"/>
-         </geometry>
-         <material name="black"/>
-      </visual>
-      <collision>
-         <origin xyz="0.011992289866897352 -0.0007726988011287212 -5.201111709052532e-06" rpy="1.5745317514920234 0.003601150001683928 1.6650413701206925"/>
-         <geometry>
-            <mesh filename="${tesollo_DG3F_file_prefix}/meshes/link_04.stl"/>
-         </geometry>
-      </collision>
-   </link>
-   <link name="F1_TIP">
-      <inertial>
-         <origin xyz="0.045 -0.000436 -7.22e-08" rpy="1.5708008179564292 -3.695361794919805e-05 1.5210948927815267"/>
-         <mass value="0.013"/>
-         <inertia ixx="1.5965708653714455e-06" iyy="1.2999999996018677e-06" izz="9.60129135026688e-07" ixy="0" ixz="0" iyz="0"/>
-      </inertial>
-      <visual>
-         <origin xyz="0.044959448417087294 -0.0004226309811080281 2.3018946871860735e-07" rpy="1.5708745579876908 -1.019986385419891e-05 1.5204133624130758"/>
-         <geometry>
-            <mesh filename="${tesollo_DG3F_file_prefix}/meshes/link_tip_high.stl"/>
-         </geometry>
-         <material name="white"/>
-      </visual>
-      <collision>
-         <origin xyz="0.044959448417087294 -0.0004226309811080281 2.3018946871860735e-07" rpy="1.5708745579876908 -1.019986385419891e-05 1.5204133624130758"/>
-         <geometry>
-            <mesh filename="${tesollo_DG3F_file_prefix}/meshes/link_tip_high.stl"/>
-         </geometry>
-      </collision>
-   </link>
-   <link name="F2_01">
-      <inertial>
-         <origin xyz="0.0003906 3.121e-08 -0.014" rpy="-0.17662368646091148 -1.9303231388878572e-06 1.5707855116626381"/>
-         <mass value="0.061"/>
-         <inertia ixx="1.924000000025899e-05" iyy="1.709411627342488e-05" izz="5.9478837263161295e-06" ixy="0" ixz="0" iyz="0"/>
-      </inertial>
-      <visual>
-         <origin xyz="0.0018977016221143523 -1.0017682763976983e-06 -0.022983822146236326" rpy="-0.1443920950720977 1.9855029389503898e-05 1.5709191233325221"/>
-         <geometry>
-            <mesh filename="${tesollo_DG3F_file_prefix}/meshes/link_01.stl"/>
-         </geometry>
-         <material name="black"/>
-      </visual>
-      <collision>
-         <origin xyz="0.0018977016221143523 -1.0017682763976983e-06 -0.022983822146236326" rpy="-0.1443920950720977 1.9855029389503898e-05 1.5709191233325221"/>
-         <geometry>
-            <mesh filename="${tesollo_DG3F_file_prefix}/meshes/link_01.stl"/>
-         </geometry>
-      </collision>
-   </link>
-   <link name="F2_02">
-      <inertial>
-         <origin xyz="0.01 3.444e-06 0.016" rpy="-0.0036890516412144943 0.31688564121750695 -0.0027736178951144786"/>
-         <mass value="0.025"/>
-         <inertia ixx="7.164797732610912e-06" iyy="6.31301833122199e-06" izz="3.274183936167101e-06" ixy="0" ixz="0" iyz="0"/>
-      </inertial>
-      <visual>
-         <origin xyz="0.010322007813576017 0.000267674195662055 0.013590600703218703" rpy="-0.03118104794815292 0.3757385725887219 -0.024334342208719002"/>
-         <geometry>
-            <mesh filename="${tesollo_DG3F_file_prefix}/meshes/link_02.stl"/>
-         </geometry>
-         <material name="black"/>
-      </visual>
-      <collision>
-         <origin xyz="0.010322007813576017 0.000267674195662055 0.013590600703218703" rpy="-0.03118104794815292 0.3757385725887219 -0.024334342208719002"/>
-         <geometry>
-            <mesh filename="${tesollo_DG3F_file_prefix}/meshes/link_02.stl"/>
-         </geometry>
-      </collision>
-   </link>
-   <link name="F2_03">
-      <inertial>
-         <origin xyz="0.014 -0.0004527 -3.953e-05" rpy="1.5651066808062148 -0.0008576993469346927 1.5562600280492769"/>
-         <mass value="0.051"/>
-         <inertia ixx="1.6912201686125405e-05" iyy="1.4940271596370447e-05" izz="6.505526717504149e-06" ixy="0" ixz="0" iyz="0"/>
-      </inertial>
-      <visual>
-         <origin xyz="0.019034639558839914 -0.0007611783816217545 0.00015734818842133856" rpy="1.5405533073968862 -0.0023628127138719535 1.5994547590929262"/>
-         <geometry>
-            <mesh filename="${tesollo_DG3F_file_prefix}/meshes/link_03.stl"/>
-         </geometry>
-         <material name="black"/>
-      </visual>
-      <collision>
-         <origin xyz="0.019034639558839914 -0.0007611783816217545 0.00015734818842133856" rpy="1.5405533073968862 -0.0023628127138719535 1.5994547590929262"/>
-         <geometry>
-            <mesh filename="${tesollo_DG3F_file_prefix}/meshes/link_03.stl"/>
-         </geometry>
-      </collision>
-   </link>
-   <link name="F2_04">
-      <inertial>
-         <origin xyz="0.012 -0.0002269 -4.676e-05" rpy="1.5668480451228681 -0.0008686188531681349 1.5829731507939977"/>
-         <mass value="0.058"/>
-         <inertia ixx="1.0860820276783573e-05" iyy="9.902070548178027e-06" izz="5.330109175038405e-06" ixy="0" ixz="0" iyz="0"/>
-      </inertial>
-      <visual>
-         <origin xyz="0.011992289866897352 -0.0007726988011287212 -5.201111709052532e-06" rpy="1.5745317514920234 0.003601150001683928 1.6650413701206925"/>
-         <geometry>
-            <mesh filename="${tesollo_DG3F_file_prefix}/meshes/link_04.stl"/>
-         </geometry>
-         <material name="black"/>
-      </visual>
-      <collision>
-         <origin xyz="0.011992289866897352 -0.0007726988011287212 -5.201111709052532e-06" rpy="1.5745317514920234 0.003601150001683928 1.6650413701206925"/>
-         <geometry>
-            <mesh filename="${tesollo_DG3F_file_prefix}/meshes/link_04.stl"/>
-         </geometry>
-      </collision>
-   </link>
-   <link name="F2_TIP">
-      <inertial>
-         <origin xyz="0.045 -0.000436 -7.22e-08" rpy="1.5708008179564292 -3.695361794919805e-05 1.5210948927815267"/>
-         <mass value="0.013"/>
-         <inertia ixx="1.5965708653714455e-06" iyy="1.2999999996018677e-06" izz="9.60129135026688e-07" ixy="0" ixz="0" iyz="0"/>
-      </inertial>
-      <visual>
-         <origin xyz="0.044959448417087294 -0.0004226309811080281 2.3018946871860735e-07" rpy="1.5708745579876908 -1.019986385419891e-05 1.5204133624130758"/>
-         <geometry>
-            <mesh filename="${tesollo_DG3F_file_prefix}/meshes/link_tip_high.stl"/>
-         </geometry>
-         <material name="white"/>
-      </visual>
-      <collision>
-      <origin xyz="0.044959448417087294 -0.0004226309811080281 2.3018946871860735e-07" rpy="1.5708745579876908 -1.019986385419891e-05 1.5204133624130758"/>
-         <geometry>
-            <mesh filename="${tesollo_DG3F_file_prefix}/meshes/link_tip_high.stl"/>
-         </geometry>
-      </collision>
-   </link>
-   <link name="F3_01">
-      <inertial>
-         <origin xyz="0.0003906 3.121e-08 -0.014" rpy="-0.17662368646091148 -1.9303231388878572e-06 1.5707855116626381"/>
-         <mass value="0.061"/>
-         <inertia ixx="1.924000000025899e-05" iyy="1.709411627342488e-05" izz="5.9478837263161295e-06" ixy="0" ixz="0" iyz="0"/>
-      </inertial>
-      <visual>
-         <origin xyz="0.0018977016221143523 -1.0017682763976983e-06 -0.022983822146236326" rpy="-0.1443920950720977 1.9855029389503898e-05 1.5709191233325221"/>
-         <geometry>
-            <mesh filename="${tesollo_DG3F_file_prefix}/meshes/link_01.stl"/>
-         </geometry>
-         <material name="black"/>
-      </visual>
-      <collision>
-      <origin xyz="0.0018977016221143523 -1.0017682763976983e-06 -0.022983822146236326" rpy="-0.1443920950720977 1.9855029389503898e-05 1.5709191233325221"/>
-         <geometry>
-            <mesh filename="${tesollo_DG3F_file_prefix}/meshes/link_01.stl"/>
-         </geometry>
-      </collision>
-   </link>
-   <link name="F3_02">
-      <inertial>
-         <origin xyz="0.01 3.444e-06 0.016" rpy="-0.0036890516412144943 0.31688564121750695 -0.0027736178951144786"/>
-         <mass value="0.025"/>
-         <inertia ixx="7.164797732610912e-06" iyy="6.31301833122199e-06" izz="3.274183936167101e-06" ixy="0" ixz="0" iyz="0"/>
-      </inertial>
-      <visual>
-         <origin xyz="0.010322007813576017 0.000267674195662055 0.013590600703218703" rpy="-0.03118104794815292 0.3757385725887219 -0.024334342208719002"/>
-         <geometry>
-            <mesh filename="${tesollo_DG3F_file_prefix}/meshes/link_02.stl"/>
-         </geometry>
-         <material name="black"/>
-      </visual>
-      <collision>
-         <origin xyz="0.010322007813576017 0.000267674195662055 0.013590600703218703" rpy="-0.03118104794815292 0.3757385725887219 -0.024334342208719002"/>
-         <geometry>
-            <mesh filename="${tesollo_DG3F_file_prefix}/meshes/link_02.stl"/>
-         </geometry>
-      </collision>
-   </link>
-   <link name="F3_03">
-      <inertial>
-         <origin xyz="0.014 -0.0004527 -3.953e-05" rpy="1.5651066808062148 -0.0008576993469346927 1.5562600280492769"/>
-         <mass value="0.051"/>
-         <inertia ixx="1.6912201686125405e-05" iyy="1.4940271596370447e-05" izz="6.505526717504149e-06" ixy="0" ixz="0" iyz="0"/>
-      </inertial>
-      <visual>
-         <origin xyz="0.019034639558839914 -0.0007611783816217545 0.00015734818842133856" rpy="1.5405533073968862 -0.0023628127138719535 1.5994547590929262"/>
-         <geometry>
-            <mesh filename="${tesollo_DG3F_file_prefix}/meshes/link_03.stl"/>
-         </geometry>
-         <material name="black"/>
-      </visual>
-      <collision>
-         <origin xyz="0.019034639558839914 -0.0007611783816217545 0.00015734818842133856" rpy="1.5405533073968862 -0.0023628127138719535 1.5994547590929262"/>
-         <geometry>
-            <mesh filename="${tesollo_DG3F_file_prefix}/meshes/link_03.stl"/>
-         </geometry>
-      </collision>
-   </link>
-   <link name="F3_04">
-      <inertial>
-         <origin xyz="0.012 -0.0002269 -4.676e-05" rpy="1.5668480451228681 -0.0008686188531681349 1.5829731507939977"/>
-         <mass value="0.058"/>
-         <inertia ixx="1.0860820276783573e-05" iyy="9.902070548178027e-06" izz="5.330109175038405e-06" ixy="0" ixz="0" iyz="0"/>
-      </inertial>
-      <visual>
-         <origin xyz="0.011992289866897352 -0.0007726988011287212 -5.201111709052532e-06" rpy="1.5745317514920234 0.003601150001683928 1.6650413701206925"/>
-         <geometry>
-            <mesh filename="${tesollo_DG3F_file_prefix}/meshes/link_04.stl"/>
-         </geometry>
-         <material name="black"/>
-      </visual>
-      <collision>
-      <origin xyz="0.011992289866897352 -0.0007726988011287212 -5.201111709052532e-06" rpy="1.5745317514920234 0.003601150001683928 1.6650413701206925"/>
-         <geometry>
-            <mesh filename="${tesollo_DG3F_file_prefix}/meshes/link_04.stl"/>
-         </geometry>
-      </collision>
-   </link>
-   <link name="F3_TIP">
-      <inertial>
-         <origin xyz="0.045 -0.000436 -7.22e-08" rpy="1.5708008179564292 -3.695361794919805e-05 1.5210948927815267"/>
-         <mass value="0.013"/>
-         <inertia ixx="1.5965708653714455e-06" iyy="1.2999999996018677e-06" izz="9.60129135026688e-07" ixy="0" ixz="0" iyz="0"/>
-      </inertial>
-      <visual>
-         <origin xyz="0.044959448417087294 -0.0004226309811080281 2.3018946871860735e-07" rpy="1.5708745579876908 -1.019986385419891e-05 1.5204133624130758"/>
-         <geometry>
-            <mesh filename="${tesollo_DG3F_file_prefix}/meshes/link_tip_high.stl"/>
-         </geometry>
-         <material name="white"/>
-      </visual>
-      <collision>
-         <origin xyz="0.044959448417087294 -0.0004226309811080281 2.3018946871860735e-07" rpy="1.5708745579876908 -1.019986385419891e-05 1.5204133624130758"/>
-         <geometry>
-            <mesh filename="${tesollo_DG3F_file_prefix}/meshes/link_tip_high.stl"/>
-         </geometry>
-      </collision>
-   </link>
-   <!--Joint -->
-   <joint name = "F1M1" type = "revolute">
-      <origin xyz="0.0265 0.0 0.0" rpy="0 0 0"/>
-      <parent link="delto_base_link"/>
-      <child link="F1_01"/>
-      <axis xyz="0.0 0.0 1.0"/>
-      <limit effort="10.0" velocity="5.0" lower="-1.0472" upper="1.0472" />
-      <dynamics damping="1.1" friction="1.1"/>
-   </joint>
-   <joint name = "F1M2" type = "revolute">
-      <origin xyz="0.0 0.0 0.0" rpy="-3.1415926207728213 -1.570796290294655 0.0"/>
-      <parent link="F1_01"/>
-      <child link="F1_02"/>
-      <axis xyz="0.0 0.0 1.0"/>
-      <limit effort="10.0" velocity="5.0" lower="-1.76278" upper="1.76278" />
-      <dynamics damping="1.1" friction="1.1"/>
-   </joint>
-   <joint name = "F1M3" type = "revolute">
-      <origin xyz="0.02022 0.0 0.03136" rpy="-1.5707963295583207 -1.5707963267948966 0.0"/>
-      <parent link="F1_02"/>
-      <child link="F1_03"/>
-      <axis xyz="0.0 0.0 1.0"/>
-      <limit effort="10.0" velocity="5.0" lower="-0.15708" upper="2.53073" />
-      <dynamics damping="1.1" friction="1.1"/>
-   </joint>
-   <joint name = "F1M4" type = "revolute">
-      <origin xyz="0.0434 0.0 0.0" rpy="0 0 0"/>
-      <parent link="F1_03"/>
-      <child link="F1_04"/>
-      <axis xyz="0.0 0.0 1.0"/>
-      <limit effort="10.0" velocity="5.0" lower="-0.226893" upper="2.02458"/>
-      <dynamics damping="1.1" friction="1.1"/>
-   </joint>
-   <joint name = "TIP1" type="fixed">
-      <origin xyz="0.0 0.0 0.0" rpy="0 0 0"/>
-      <parent link="F1_04"/>
-      <child link="F1_TIP"/>
-   </joint>
-   <!-- FINGER 2-->
-   <joint name = "F2M1" type = "revolute">
-      <origin xyz="-0.01334 0.023 0.0" rpy="0 0 -3.14"/>
-      <parent link="delto_base_link"/>
-      <child link="F2_01"/>
-      <axis xyz="0.0 0.0 1.0"/>
-      <limit effort="10.0" velocity="5.0" lower="-1.91986" upper="0.139626" />
-      <dynamics damping="1.1" friction="1.1"/>
-   </joint>
-   <joint name = "F2M2" type = "revolute">
-      <origin xyz="0.0 0.0 0.0" rpy="-3.14 -1.57 0"/>
-      <parent link="F2_01"/>
-      <child link="F2_02"/>
-      <axis xyz="0.0 0.0 1.0"/>
-      <limit effort="10.0" velocity="5.0" lower="-1.76278" upper="1.76278" />
-      <dynamics damping="1.1" friction="1.1"/>
-   </joint>
-   <joint name = "F2M3" type = "revolute">
-      <origin xyz="0.02022 0.0 0.03136" rpy="-1.57 -1.57 0"/>
-      <parent link="F2_02"/>
-      <child link="F2_03"/>
-      <axis xyz="0.0 0.0 1.0"/>
-      <limit effort="10.0" velocity="5.0" lower="-0.15708" upper="2.53073" />
-      <dynamics damping="1.1" friction="1.1"/>
-   </joint>
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