Commit message: Fixed tesollo oreinetation bug

File: libs/robot_description/composites/panda_w_tesollo.urdf.xacro (robot description, xacro)
@@ -15,9 +15,8 @@
     <xacro:tesollo_DG3F name_prefix="${name_prefix}" file_prefix="${tesollo_DG3F_file_prefix}"/>
     <!-- Connection Joints -->
-    <!-- TODO: Check rotation and height -->
     <joint name="${name_prefix}panda_gripper_joint" type="fixed">
       <parent link="${name_prefix}panda_link8"/>
       <child link="${name_prefix}delto_base_link"/>
-      <origin rpy="0 0 0" xyz="0 0 0.106"/>
+      <origin rpy="0 0 -0.785" xyz="0 0 0.106"/>
     </joint>
   </xacro:macro>

File: libs/robot_description/ros/bimanual_arms.urdf (robot description, URDF)
Before this commit: robot bimanual_arms, 54 links, 53 joints
Joints:
- joint left_panda_gripper_joint: origin xyz=0 0 0.106 rpy=0 0 0 -> xyz=0 0 0.106 rpy=0 0 -0.785
- joint right_F1M4: origin xyz=0.0 0.0 0.0 rpy=0 0 0 -> xyz=0.0434 0.0 0.0 rpy=0 0 0
- joint right_F2M4: axis 0.0434 0.0 1.0 -> 0.0 0.0 1.0
- joint right_panda_gripper_joint: origin xyz=0 0 0.106 rpy=0 0 0 -> xyz=0 0 0.106 rpy=0 0 -0.785

File: libs/robot_description/tesollo_DG3F/tesollo_DG3F.urdf.xacro (robot description, xacro)
@@ -451,4 +451,11 @@
             <child link="${name_prefix}F3_TIP"/>
         </joint>
+        <!-- "Middle" of grasp -->
+        <link name="${name_prefix}delto_offset_link"/>
+        <joint name="${name_prefix}delto_offset_joint" type="fixed">
+            <parent link="${name_prefix}delto_base_link"/>
+            <child  link="${name_prefix}delto_offset_link"/>
+            <origin xyz="0 0 0.05" rpy="0 0 0"/>
+        </joint>
     </xacro:macro>
 </robot>
