Commit message: attempting to add fingers into rangedik

File: libs/robot_description/ros/bimanual_arms.urdf (robot description, URDF)
Before this commit: robot bimanual_arms, 52 links, 51 joints
Joints:
- joint left_F2M4: axis 0.0434 0.0 1.0 -> 0.0 0.0 1.0

Commit message: added to multi_chain_ranged_ik.py for 2 arm IK as well as changes in bimanual_arms.urdf for invisible link in front of palm

File: libs/robot_description/ros/bimanual_arms.urdf (robot description, URDF)
Before this commit: robot bimanual_arms, 52 links, 51 joints
Links:
- added link left_delto_offset_link
- added link right_delto_offset_link
Joints:
- added joint left_delto_offset_joint: type fixed, parent left_delto_base_link, child left_delto_offset_link, origin xyz=0 0 0.05 rpy=0 0 0
- added joint right_delto_offset_joint: type fixed, parent right_delto_base_link, child right_delto_offset_link, origin xyz=0 0 0.05 rpy=0 0 0
