Commit message: made some changes, commiting before regenerating xacro

File: libs/robot_description/ros/src/robot_description/urdf/composites/bimanual_arms.urdf.xacro (robot description, xacro)
@@ -1,23 +1,28 @@
 <?xml version="1.0" encoding="utf-8"?>
-<robot  name="bimanual_arms" xmlns:xacro="http://www.ros.org/wiki/xacro">
-  <xacro:arg name="composite_file_prefix"  default="package://robot_description/composites"/>
-  <xacro:arg name="panda_file_prefix"  default="package://robot_description/panda"/>
-  <xacro:arg name="tesollo_DG3F_file_prefix"  default="package://robot_description/tesollo"/>
+<robot  name="${name_prefix}bimanual_arms" xmlns:xacro="http://www.ros.org/wiki/xacro">
+  <xacro:arg name="name_prefix" default=""/>
+  <xacro:arg name="composite_file_prefix" default="package://robot_description/composites"/>
+  <xacro:arg name="panda_file_prefix" default="package://robot_description/panda"/>
+  <xacro:arg name="tesollo_DG3F_file_prefix" default="package://robot_description/tesollo"/>
   <xacro:include filename="$(arg composite_file_prefix)/panda_w_tesollo.urdf.xacro"/>
-  <xacro:panda_w_tesollo name_prefix="left_" panda_file_prefix="$(arg panda_file_prefix)"
-                 tesollo_DG3F_file_prefix="$(arg tesollo_DG3F_file_prefix)"/>
-  <xacro:panda_w_tesollo name_prefix="right_" panda_file_prefix="$(arg panda_file_prefix)"
-                 tesollo_DG3F_file_prefix="$(arg tesollo_DG3F_file_prefix)"/>
-  <!-- Connection Joints -->
-  <joint name="left_panda_mount" type="fixed">
-    <parent link="table_top"/>
-    <child link="left_panda_link0"/>
-    <origin rpy="0 0 0" xyz="-0.558 -0.092 0.0225"/>
-  </joint>
-  <joint name="right_panda_mount" type="fixed">
-    <parent link="table_top"/>
-    <child link="right_panda_link0"/>
-    <origin rpy="0 0 3.14" xyz="0.5588 -0.092 0.0225"/>
-  </joint>
+  <xacro:panda_w_tesollo
+    name_prefix="${name_prefix}left_"
+    panda_file_prefix="$(arg panda_file_prefix)"
+    tesollo_DG3F_file_prefix="$(arg tesollo_DG3F_file_prefix)"/>
+  <xacro:panda_w_tesollo
+    name_prefix="${name_prefix}right_"
+    panda_file_prefix="$(arg panda_file_prefix)"
+    tesollo_DG3F_file_prefix="$(arg tesollo_DG3F_file_prefix)"/>
+    <!-- Connection Joints -->
+    <joint name="${name_prefix}left_panda_mount" type="fixed">
+      <parent link="table_top"/>
+      <child link="${name_prefix}left_panda_link0"/>
+      <origin rpy="0 0 0" xyz="-0.558 -0.092 0.0225"/>
+    </joint>
+    <joint name="${name_prefix}right_panda_mount" type="fixed">
+      <parent link="table_top"/>
+      <child link="${name_prefix}right_panda_link0"/>
+      <origin rpy="0 0 3.14" xyz="0.5588 -0.092 0.0225"/>
+    </joint>
   <!-- TABLE -->
   <link name="table"/>

Commit message: added the offset link and changed some type handling in reset in ranged_ik.py

File: libs/robot_description/ros/src/robot_description/urdf/composites/bimanual_arms.urdf.xacro (robot description, xacro)
@@ -1,4 +1,4 @@
 <?xml version="1.0" encoding="utf-8"?>
-<robot  name="${name_prefix}bimanual_arms" xmlns:xacro="http://www.ros.org/wiki/xacro">
+<robot  name="$(arg name_prefix)bimanual_arms" xmlns:xacro="http://www.ros.org/wiki/xacro">
   <xacro:arg name="name_prefix" default=""/>
   <xacro:arg name="composite_file_prefix" default="package://robot_description/composites"/>
@@ -7,20 +7,20 @@
   <xacro:include filename="$(arg composite_file_prefix)/panda_w_tesollo.urdf.xacro"/>
   <xacro:panda_w_tesollo
-    name_prefix="${name_prefix}left_"
+    name_prefix="$(arg name_prefix)left_"
     panda_file_prefix="$(arg panda_file_prefix)"
     tesollo_DG3F_file_prefix="$(arg tesollo_DG3F_file_prefix)"/>
   <xacro:panda_w_tesollo
-    name_prefix="${name_prefix}right_"
+    name_prefix="$(arg name_prefix)right_"
     panda_file_prefix="$(arg panda_file_prefix)"
     tesollo_DG3F_file_prefix="$(arg tesollo_DG3F_file_prefix)"/>
     <!-- Connection Joints -->
-    <joint name="${name_prefix}left_panda_mount" type="fixed">
+    <joint name="$(arg name_prefix)left_panda_mount" type="fixed">
       <parent link="table_top"/>
-      <child link="${name_prefix}left_panda_link0"/>
+      <child link="$(arg name_prefix)left_panda_link0"/>
       <origin rpy="0 0 0" xyz="-0.558 -0.092 0.0225"/>
     </joint>
-    <joint name="${name_prefix}right_panda_mount" type="fixed">
+    <joint name="$(arg name_prefix)right_panda_mount" type="fixed">
       <parent link="table_top"/>
-      <child link="${name_prefix}right_panda_link0"/>
+      <child link="$(arg name_prefix)right_panda_link0"/>
       <origin rpy="0 0 3.14" xyz="0.5588 -0.092 0.0225"/>
     </joint>

File: libs/robot_description/ros/src/robot_description/urdf/panda/panda.urdf.xacro (robot description, xacro)
@@ -1,4 +1,5 @@
 <?xml version="1.0" encoding="utf-8"?>
 <robot xmlns:xacro="http://www.ros.org/wiki/xacro">
+  <xacro:arg name="name_prefix" default=""/>
   <xacro:macro name="panda" params="file_prefix:='package://robot_description/panda' name_prefix:=''">
     <link name="${name_prefix}panda_link0">

File: libs/robot_description/ros/src/robot_description/urdf/panda/panda_hand.urdf.xacro (robot description, xacro)
@@ -1,4 +1,5 @@
 <?xml version="1.0" encoding="utf-8"?>
 <robot xmlns:xacro="http://www.ros.org/wiki/xacro">
+  <xacro:arg name="name_prefix" default=""/>
   <xacro:macro name="panda_hand" params="file_prefix:='package://robot_description/panda' name_prefix:=''">
     <link name="${name_prefix}panda_hand">

File: libs/robot_description/ros/src/robot_description/urdf/tesollo_DG3F/tesollo_DG3F.urdf.xacro (robot description, xacro)
@@ -10,5 +10,6 @@
 -->
 <robot xmlns:xacro="http://www.ros.org/wiki/xacro">
-   <xacro:macro name="tesollo_DG3F" params="file_prefix:='package://robot_description/tesollo_DG3F' name_prefix:='' ">
+    <xacro:arg name="name_prefix" default=""/>
+    <xacro:macro name="tesollo_DG3F" params="file_prefix:='package://robot_description/tesollo_DG3F' name_prefix:='' ">
         <material name="${name_prefix}black">
             <color rgba="0.196 0.196 0.196 1.0"/>
@@ -37,4 +38,10 @@
             </collision>
         </link>
+        <link name="${name_prefix}delto_offset_link"/>
+        <joint name="${name_prefix}delto_offset_joint" type="fixed">
+          <parent link="${name_prefix}delto_base_link"/>
+          <child link="${name_prefix}delto_offset_link"/>
+          <origin xyz="0 0 0.05" rpy="0 0 0"/>
+        </joint>
         <link name="${name_prefix}F1_01">
             <inertial>
