Commit message: deleted duplicate delto_base_offset in tesollo_DG3F.urdf.xacro

File: libs/robot_description/ros/src/robot_description/urdf/tesollo_DG3F/tesollo_DG3F.urdf.xacro (robot description, xacro)
@@ -457,11 +457,4 @@
             <child link="${name_prefix}F3_TIP"/>
         </joint>
-        <!-- "Middle" of grasp -->
-        <link name="${name_prefix}delto_offset_link"/>
-        <joint name="${name_prefix}delto_offset_joint" type="fixed">
-            <parent link="${name_prefix}delto_base_link"/>
-            <child  link="${name_prefix}delto_offset_link"/>
-            <origin xyz="0 0 0.05" rpy="0 0 0"/>
-        </joint>
     </xacro:macro>
 </robot>
