Commit message: Adjust gripper position in urdf and usd but still need to update friction

File: libs/robot_description/ros/src/robot_description/urdf/bimanual_arms.urdf (robot description, URDF)
Before this commit: robot bimanual_arms, 54 links, 53 joints
Joints:
- joint left_panda_gripper_joint: origin xyz=0 0 0.106 rpy=0 0 -0.785 -> xyz=0 0 0.106 rpy=0 0 -1.015
- joint right_panda_gripper_joint: origin xyz=0 0 0.106 rpy=0 0 -0.785 -> xyz=0 0 0.106 rpy=0 0 -1.015

File: libs/robot_description/ros/src/robot_description/urdf/composites/panda_w_tesollo.urdf.xacro (robot description, xacro)
@@ -20,5 +20,5 @@
       <parent link="${name_prefix}panda_link8"/>
       <child link="${name_prefix}delto_base_link"/>
-      <origin rpy="0 0 -0.785" xyz="0 0 0.106"/>
+      <origin rpy="0 0 -1.015" xyz="0 0 0.106"/>
     </joint>
   </xacro:macro>
