Commit message: Cleaned up mujuco

File: libs/robot_description/ros/src/robot_description/urdf/panda/panda.urdf.xacro (robot description, xacro)
@@ -44,4 +44,5 @@
       <axis xyz="0 0 1"/>
       <limit effort="87" lower="-2.8973" upper="2.8973" velocity="2.1750"/>
+      <dynamics damping="5.0" friction="0.0"/>
     </joint>
     <link name="${name_prefix}panda_link2">
@@ -70,4 +71,5 @@
       <axis xyz="0 0 1"/>
       <limit effort="87" lower="-1.7628" upper="1.7628" velocity="2.1750"/>
+      <dynamics damping="5.0" friction="0.0"/>
     </joint>
     <link name="${name_prefix}panda_link3">
@@ -96,4 +98,5 @@
       <axis xyz="0 0 1"/>
       <limit effort="87" lower="-2.8973" upper="2.8973" velocity="2.1750"/>
+      <dynamics damping="5.0" friction="0.0"/>
     </joint>
     <link name="${name_prefix}panda_link4">
@@ -122,4 +125,5 @@
       <axis xyz="0 0 1"/>
       <limit effort="87" lower="-3.0718" upper="-0.0698" velocity="2.1750"/>
+      <dynamics damping="5.0" friction="0.0"/>
     </joint>
     <link name="${name_prefix}panda_link5">
@@ -148,4 +152,5 @@
       <axis xyz="0 0 1"/>
       <limit effort="12" lower="-2.8973" upper="2.8973" velocity="2.6100"/>
+      <dynamics damping="5.0" friction="0.0"/>
     </joint>
     <link name="${name_prefix}panda_link6">
@@ -174,4 +179,5 @@
       <axis xyz="0 0 1"/>
       <limit effort="12" lower="-0.0175" upper="3.7525" velocity="2.6100"/>
+      <dynamics damping="5.0" friction="0.0"/>
     </joint>
     <link name="${name_prefix}panda_link7">
@@ -200,4 +206,5 @@
       <axis xyz="0 0 1"/>
       <limit effort="12" lower="-2.8973" upper="2.8973" velocity="2.6100"/>
+      <dynamics damping="5.0" friction="0.0"/>
     </joint>
     <link name="${name_prefix}panda_link8"/>
